File: basic_microcontroller.kicad_sch (KiCad schematic)
At the start: 81 parts, among them J1 USB_C_Receptacle_USB2.0, J2 AVR-ISP-6, J3 Screw_Terminal_01x02, U1 ATmega32U4-A, Y1 8MHz

Commit message: Fixed wiring on button
Connections:
- net GND: now also S1.4 (COM_2); no longer S1.1 (COM_1), S1.3 (NC_1)
- net RESET: now also S1.5 (NO_2); no longer S1.4 (COM_2), S1.6 (NC_2)
- no-connect marks 6 -> 8
Changed lines of the file:
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@@
   (junction (at 69.215 168.91) (diameter 0) (color 0 0 0 0)
   )
-  (junction (at 48.895 48.26) (diameter 0) (color 0 0 0 0)
-  )
   (junction (at 256.54 119.38) (diameter 0) (color 0 0 0 0)
   )
@@
   )
   (junction (at 237.49 27.94) (diameter 0) (color 0 0 0 0)
-  )
-  (junction (at 84.455 48.26) (diameter 0) (color 0 0 0 0)
   )
   (junction (at 93.345 60.96) (diameter 0) (color 0 0 0 0)
@@
   (no_connect (at 50.165 105.41))
   (no_connect (at 137.795 82.55))
+  (no_connect (at 51.435 45.72))
   (no_connect (at 137.795 80.01))
-  (no_connect (at 81.915 48.26))
+  (no_connect (at 81.915 50.8))
+  (no_connect (at 51.435 50.8))
   (no_connect (at 50.165 107.95))
   (wire (pts (xy 70.485 64.77) (xy 74.295 64.77))
@@
     (stroke (width 0) (type default))
   )
-  (wire (pts (xy 95.885 48.26) (xy 95.885 57.15))
-    (stroke (width 0) (type default))
-  )
   (wire (pts (xy 195.58 81.28) (xy 195.58 83.82))
     (stroke (width 0) (type default))
@@
     (stroke (width 0) (type default))
   )
-  (wire (pts (xy 81.915 50.8) (xy 84.455 50.8))
-    (stroke (width 0) (type default))
-  )
   (wire (pts (xy 256.54 81.28) (xy 256.54 83.82))
     (stroke (width 0) (type default))
@@
     (stroke (width 0) (type default))
   )
-  (wire (pts (xy 48.895 48.26) (xy 48.895 45.72))
-    (stroke (width 0) (type default))
-  )
   (wire (pts (xy 106.68 173.99) (xy 107.95 173.99))
     (stroke (width 0) (type default))
@@
     (stroke (width 0) (type default))
   )
+  (wire (pts (xy 95.885 57.15) (xy 95.885 48.26))
+    (stroke (width 0) (type default))
+  )
   (wire (pts (xy 237.49 27.94) (xy 256.54 27.94))
     (stroke (width 0) (type default))
   )
-  (wire (pts (xy 84.455 50.8) (xy 84.455 48.26))
-    (stroke (width 0) (type default))
-  )
   (wire (pts (xy 122.555 44.45) (xy 122.555 41.91))
     (stroke (width 0) (type default))
@@
     (stroke (width 0) (type default))
   )
-  (wire (pts (xy 48.895 45.72) (xy 51.435 45.72))
-    (stroke (width 0) (type default))
-  )
   (wire (pts (xy 103.505 82.55) (xy 107.315 82.55))
     (stroke (width 0) (type default))
@@
     (stroke (width 0) (type default))
   )
+  (wire (pts (xy 81.915 38.735) (xy 88.265 38.735))
+    (stroke (width 0) (type default))
+  )
   (wire (pts (xy 121.285 143.51) (xy 121.285 147.32))
     (stroke (width 0) (type default))
@@
     (stroke (width 0) (type default))
   )
-  (wire (pts (xy 42.545 50.8) (xy 42.545 48.26))
-    (stroke (width 0) (type default))
-  )
   (wire (pts (xy 22.225 53.975) (xy 22.225 47.625))
     (stroke (width 0) (type default))
@@
     (stroke (width 0) (type default))
   )
-  (wire (pts (xy 48.895 50.8) (xy 48.895 48.26))
-    (stroke (width 0) (type default))
-  )
   (wire (pts (xy 256.54 139.7) (xy 256.54 137.16))
     (stroke (width 0) (type default))
@@
     (stroke (width 0) (type default))
   )
-  (wire (pts (xy 42.545 48.26) (xy 48.895 48.26))
-    (stroke (width 0) (type default))
-  )
   (wire (pts (xy 190.5 119.38) (xy 195.58 119.38))
     (stroke (width 0) (type default))
@@
     (stroke (width 0) (type default))
   )
-  (wire (pts (xy 81.915 45.72) (xy 84.455 45.72))
-    (stroke (width 0) (type default))
-  )
   (wire (pts (xy 95.885 72.39) (xy 107.315 72.39))
     (stroke (width 0) (type default))
@@
     (stroke (width 0) (type default))
   )
+  (wire (pts (xy 81.915 45.72) (xy 81.915 38.735))
+    (stroke (width 0) (type default))
+  )
   (wire (pts (xy 157.48 137.795) (xy 157.48 141.605))
     (stroke (width 0) (type default))
@@
     (stroke (width 0) (type default))
   )
-  (wire (pts (xy 84.455 48.26) (xy 95.885 48.26))
-    (stroke (width 0) (type default))
-  )
   (wire (pts (xy 51.435 82.55) (xy 50.165 82.55))
     (stroke (width 0) (type default))
@@
     (stroke (width 0) (type default))
   )
-  (wire (pts (xy 51.435 50.8) (xy 48.895 50.8))
-    (stroke (width 0) (type default))
-  )
   (wire (pts (xy 215.9 48.26) (xy 215.9 45.72))
     (stroke (width 0) (type default))
@@
     (stroke (width 0) (type default))
   )
+  (wire (pts (xy 81.915 48.26) (xy 95.885 48.26))
+    (stroke (width 0) (type default))
+  )
   (wire (pts (xy 256.54 71.12) (xy 256.54 68.58))
     (stroke (width 0) (type default))
@@
   )
   (wire (pts (xy 256.54 104.14) (xy 256.54 106.68))
-    (stroke (width 0) (type default))
-  )
-  (wire (pts (xy 84.455 45.72) (xy 84.455 48.26))
     (stroke (width 0) (type default))
   )
@@
     )
   )
-  (symbol (lib_id "power:GND") (at 42.545 50.8 0) (unit 1)
+  (symbol (lib_id "power:GND") (at 88.265 38.735 0) (unit 1)
     (in_bom yes) (on_board yes) (dnp no) (fields_autoplaced)
-    (property "Reference" "#PWR014" (at 42.545 57.15 0)
-      (effects (font (size 1.27 1.27)) hide)
-    )
-    (property "Value" "GND" (at 42.545 55.88 0)
+    (property "Reference" "#PWR014" (at 88.265 45.085 0)
+      (effects (font (size 1.27 1.27)) hide)
+    )
+    (property "Value" "GND" (at 88.265 43.815 0)
       (effects (font (size 1.27 1.27)))
     )
-    (property "Footprint" "" (at 42.545 50.8 0)
-      (effects (font (size 1.27 1.27)) hide)
-    )
-    (property "Datasheet" "" (at 42.545 50.8 0)
-      (effects (font (size 1.27 1.27)) hide)
-    )
+    (property "Footprint" "" (at 88.265 38.735 0)
+      (effects (font (size 1.27 1.27)) hide)
+    )
+    (property "Datasheet" "" (at 88.265 38.735 0)
+      (effects (font (size 1.27 1.27)) hide)
+    )
